Commit message: adding base for whycon marker

File: rotors_description/urdf/crazyflie2.xacro (robot description, xacro)
@@ -38,4 +38,7 @@
   <xacro:property name="rotor_drag_coefficient" value="8.06428e-05" />
   <xacro:property name="rolling_moment_coefficient" value="0.000001" />
+<!--   <xacro:property name="marker" value="whycon_marker" />
+  <xacro:property name="marker_radius" value="0.08"/>
+  <xacro:property name="marker_width" value="0.005"/>  -->
   <!-- Property Blocks -->
   <xacro:property name="body_inertia">

File: rotors_description/urdf/crazyflie2_base.xacro (robot description, xacro)
@@ -19,4 +19,6 @@
   <!-- Instantiate crazyflie2 "mechanics" -->
   <xacro:include filename="$(find rotors_description)/urdf/crazyflie2.xacro" />
+  <!-- To call file containing information about whycon_marker base's description -->
+  <xacro:include filename="$(find rotors_description)/urdf/whycon_marker_file.xacro"/>
   <!-- Instantiate a controller. -->
   <xacro:controller_plugin_macro namespace="${namespace}" imu_sub_topic="imu" />
@@ -43,3 +45,5 @@
       rotor_velocity_slowdown_sim="${rotor_velocity_slowdown_sim}" />
   </xacro:if>
+  <!-- To mount a whycon_marker base -->
+  <xacro:whycon_marker namespace="${namespace}" marker="whycon_marker" marker_width="0.001" marker_radius="0.025"/>
 </robot>
